File: PCB_Project/encoder_protyping_board/encoder_protyping_board.kicad_pcb (KiCad board)
At the start: 2 copper layers, 22 x 21.6 mm, 13 parts, among them J1 Conn_02x04_Counter_Clockwise, J2 Conn_01x02_Pin, J3 Conn_01x03_Pin

Commit message: slightly sorter ground path to U1
Routing:
- net GND: vias 18 -> 19
Changed lines of the file:
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@@
   (segment (start 71.643 15.494) (end 69.992 17.145) (width 0.25) (layer "F.Cu") (net 2))
   (segment (start 68.58 25.4) (end 68.58 24.542462) (width 0.25) (layer "F.Cu") (net 2))
-  (segment (start 57.521 31.1558) (end 57.521 26.431) (width 0.25) (layer "F.Cu") (net 2))
+  (segment (start 57.521 31.1558) (end 57.521 27.4728) (width 0.25) (layer "F.Cu") (net 2))
+  (segment (start 57.521 27.4728) (end 57.5056 27.4574) (width 0.25) (layer "F.Cu") (net 2))
   (segment (start 68.58 24.542462) (end 71.755 21.367462) (width 0.25) (layer "F.Cu") (net 2))
+  (segment (start 57.5056 27.4574) (end 57.521 27.442) (width 0.25) (layer "F.Cu") (net 2))
   (segment (start 68.58 25.4) (end 68.707 25.4) (width 0.25) (layer "F.Cu") (net 2))
   (segment (start 71.501 34.925) (end 76.2 34.925) (width 0.25) (layer "F.Cu") (net 2))
@@
   (segment (start 70.675 25.4) (end 71.13 25.4) (width 0.25) (layer "F.Cu") (net 2))
   (segment (start 69.992 17.145) (end 68.817 15.97) (width 0.25) (layer "F.Cu") (net 2))
+  (segment (start 57.521 27.442) (end 57.521 26.431) (width 0.25) (layer "F.Cu") (net 2))
   (segment (start 65.183 18.32) (end 68.817 18.32) (width 0.25) (layer "F.Cu") (net 2))
   (segment (start 71.755 21.367462) (end 71.755 19.583701) (width 0.25) (layer "F.Cu") (net 2))
@@
   (via (at 71.1708 36.3728) (size 0.8) (drill 0.4) (layers "F.Cu" "B.Cu") (free) (net 2))
   (via (at 73.8124 21.2598) (size 0.8) (drill 0.4) (layers "F.Cu" "B.Cu") (free) (net 2))
+  (via (at 57.5056 27.4574) (size 0.8) (drill 0.4) (layers "F.Cu" "B.Cu") (net 2))
   (via (at 69.3166 20.4978) (size 0.8) (drill 0.4) (layers "F.Cu" "B.Cu") (free) (net 2))
   (via (at 62.865 29.337) (size 0.8) (drill 0.4) (layers "F.Cu" "B.Cu") (free) (net 2))

Commit message: added jumper setting on rear silkscreen
Parts:
- JP1: footprint Jumper:SolderJumper-3_P1.3mm_Open_RoundedPad1.0x1.5mm -> Jumper:SolderJumper-3_P1.3mm_Open_RoundedPad1.0x1.5mm_NumberLabels
Other:
- board text added: "↑↑ 0x58 ↑↓ 0x5A ↓↑ 0x5C ↓↓ 0x5E"
Changed lines of the file:
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@@
     )
   )
-  (footprint "Jumper:SolderJumper-3_P1.3mm_Open_RoundedPad1.0x1.5mm" (layer "B.Cu")
-    (at 61.625 18.216 90)
-    (descr "SMD Solder 3-pad Jumper, 1x1.5mm rounded Pads, 0.3mm gap, open")
+  (footprint "Jumper:SolderJumper-3_P1.3mm_Open_RoundedPad1.0x1.5mm_NumberLabels" (layer "B.Cu")
+    (at 61.595 18.191 90)
+    (descr "SMD Solder 3-pad Jumper, 1x1.5mm rounded Pads, 0.3mm gap, open, labeled with numbers")
     (tags "solder jumper open")
     (property "Sheetfile" "encoder_protyping_board.kicad_sch")
@@
     (property "ki_keywords" "Solder Jumper SPDT")
     (attr exclude_from_pos_files)
-    (fp_text reference "JP1" (at 7.717 3.404 90) (layer "B.SilkS")
+    (fp_text reference "JP1" (at 0 1.8 270) (layer "B.SilkS") hide
         (effects (font (size 1 1) (thickness 0.15)) (justify mirror))
     )
-    (fp_text value "SolderJumper_3_Open" (at 0 -1.9 90) (layer "B.Fab") hide
+    (fp_text value "SolderJumper_3_Open" (at -3.3486 24.0284 270) (layer "B.Fab") hide
         (effects (font (size 1 1) (thickness 0.15)) (justify mirror))
     )
     (fp_line (start -2.05 -0.3) (end -2.05 0.3)
       (stroke (width 0.12) (type solid)) (layer "B.SilkS"))
-    (fp_line (start -1.5 -1.5) (end -0.9 -1.5)
-      (stroke (width 0.12) (type solid)) (layer "B.SilkS"))
     (fp_line (start -1.4 1) (end 1.4 1)
-      (stroke (width 0.12) (type solid)) (layer "B.SilkS"))
-    (fp_line (start -1.2 -1.2) (end -1.5 -1.5)
-      (stroke (width 0.12) (type solid)) (layer "B.SilkS"))
-    (fp_line (start -1.2 -1.2) (end -0.9 -1.5)
       (stroke (width 0.12) (type solid)) (layer "B.SilkS"))
     (fp_line (start 1.4 -1) (end -1.4 -1)
@@
   (gr_rect (start 56.134 15.24) (end 78.105 36.83)
     (stroke (width 0.1) (type default)) (fill none) (layer "Edge.Cuts"))
+  (gr_text "↑↑ 0x58\n↑↓ 0x5A\n↓↑ 0x5C\n↓↓ 0x5E" (at 64.0588 27.051) (layer "B.SilkS")
+    (effects (font (size 1 1) (thickness 0.15)) (justify left bottom mirror))
+  )
   (segment (start 58.4454 27.723) (end 58.4454 30.1401) (width 0.25) (layer "F.Cu") (net 1))
   (segment (start 58.4434 27.725) (end 58.4454 27.723) (width 0.25) (layer "F.Cu") (net 1))

Commit message: Labeled part values
Parts:
- C 10nf: renamed from C2
- C 4.7μF: renamed from C3
- C 4.7μF: renamed from C1
- R 1.2k: renamed from R1
- R 1.6k: renamed from R2
- R 1.6k: renamed from R3
- renumbered U2 to A3903, U1 to PCA9629A
Changed lines of the file:
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@@
     (property "Sheetname" "")
     (attr smd)
-    (fp_text reference "U2" (at 0 -3.5) (layer "F.SilkS")
+    (fp_text reference "A3903" (at 0 -3.5) (layer "F.SilkS")
         (effects (font (size 1 1) (thickness 0.15)))
     )
@@
     (property "ki_keywords" "R res resistor")
     (attr smd)
-    (fp_text reference "R1" (at 2.286 0 180) (layer "F.SilkS")
+    (fp_text reference "R 1.2k" (at 3.5286 0 180) (layer "F.SilkS")
         (effects (font (size 1 1) (thickness 0.15)))
     )
@@
     (property "ki_keywords" "cap capacitor")
     (attr through_hole)
-    (fp_text reference "C3" (at 0.955112 3.81) (layer "F.SilkS")
+    (fp_text reference "C 4.7μF" (at 0.955112 3.81) (layer "F.SilkS")
         (effects (font (size 1 1) (thickness 0.15)))
     )
@@
     (property "Sheetname" "")
     (attr smd)
-    (fp_text reference "U1" (at 0 -3.45) (layer "F.SilkS")
+    (fp_text reference "PCA9629A" (at 0 -3.45) (layer "F.SilkS")
         (effects (font (size 1 1) (thickness 0.15)))
     )
@@
     (property "ki_keywords" "cap capacitor")
     (attr smd)
-    (fp_text reference "C2" (at 0 1.27) (layer "F.SilkS")
+    (fp_text reference "C 10nf" (at -4.79838 -1.397) (layer "F.SilkS")
         (effects (font (size 1 1) (thickness 0.15)))
     )
@@
     (property "ki_keywords" "cap capacitor")
     (attr smd)
-    (fp_text reference "C1" (at 0 -1.524) (layer "F.SilkS")
+    (fp_text reference "C 4.7μF" (at -4.346 -1.3716) (layer "F.SilkS")
         (effects (font (size 1 1) (thickness 0.15)))
     )
@@
     (property "ki_keywords" "R res resistor")
     (attr smd)
-    (fp_text reference "R2" (at -2.286 -0.254) (layer "F.SilkS")
+    (fp_text reference "R 1.6k" (at -3.5363 -0.254) (layer "F.SilkS")
         (effects (font (size 1 1) (thickness 0.15)))
     )
@@
     (property "ki_keywords" "R res resistor")
     (attr smd)
-    (fp_text reference "R3" (at 2.2683 0.3302) (layer "F.SilkS")
-        (effects (font (size 1 1) (thickness 0.15)))
-    )
+    (fp_text reference "R 1.6k" (at 3.5383 0.3302) (layer "F.SilkS")
+        (effects (font (size 1 1) (thickness 0.15)))
+    )
