File: PCB_Project/encoder_protyping_board/encoder_protyping_board.kicad_sch (KiCad schematic)
At the start: 13 parts, among them J1 Conn_02x04_Counter_Clockwise, J2 Conn_01x02_Pin, J3 Conn_01x03_Pin

Commit message: added jumper setting on rear silkscreen
Parts:
- JP1: footprint Jumper:SolderJumper-3_P1.3mm_Open_RoundedPad1.0x1.5mm -> Jumper:SolderJumper-3_P1.3mm_Open_RoundedPad1.0x1.5mm_NumberLabels
Changed lines of the file:
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@@
       (effects (font (size 1.27 1.27)) (justify left))
     )
-    (property "Footprint" "Jumper:SolderJumper-3_P1.3mm_Open_RoundedPad1.0x1.5mm" (at 74.93 71.12 0)
+    (property "Footprint" "Jumper:SolderJumper-3_P1.3mm_Open_RoundedPad1.0x1.5mm_NumberLabels" (at 74.93 71.12 0)
       (effects (font (size 1.27 1.27)) hide)
     )

Commit message: Labeled part values
Parts:
- JP1: footprint Jumper:SolderJumper-3_P1.3mm_Open_RoundedPad1.0x1.5mm_NumberLabels -> Jumper:SolderJumper-3_P1.3mm_Open_RoundedPad1.0x1.5mm
Changed lines of the file:
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@@
       (effects (font (size 1.27 1.27)) (justify left))
     )
-    (property "Footprint" "Jumper:SolderJumper-3_P1.3mm_Open_RoundedPad1.0x1.5mm_NumberLabels" (at 74.93 71.12 0)
+    (property "Footprint" "Jumper:SolderJumper-3_P1.3mm_Open_RoundedPad1.0x1.5mm" (at 74.93 71.12 0)
       (effects (font (size 1.27 1.27)) hide)
     )
