File: PCB_Project/power_management.kicad_sch (KiCad schematic)
At the start: 20 parts, among them J6 Batt_Connector, U10 LM22678TJ-5, U9 LM22678TJ-ADJ

Commit message: power distribution done
Parts:
- removed C14, C19: C_Polarized, symbol Device:C_Polarized_US
- removed C17: 180µF, symbol Device:C_Polarized_US
- removed C21: C, symbol Device:C
- removed C22: C, symbol Device:C_Polarized_US
- removed D1, D2: D_Schottky, symbol Device:D_Schottky
- removed J6: Batt_Connector, Connector_JST:JST_PH_B2B-PH-K_1x02_P2.00mm_Vertical, symbol Connector:Conn_01x02_Socket
- removed U10: LM22678TJ-5, Package_TO_SOT_SMD:TO-263-7_TabPin8, symbol Regulator_Switching:LM22678TJ-5
- removed U9: LM22678TJ-ADJ, Package_TO_SOT_SMD:TO-263-7_TabPin8, symbol Regulator_Switching:LM22678TJ-ADJ
- added C14, C39, C40, C45, C46: 100nF, Capacitor_SMD:C_0402_1005Metric, symbol Device:C
- added C17, C19, C41, C47: 10µF, Capacitor_SMD:C_0402_1005Metric, symbol Device:C
- added C21, C22, C23, C24, C43, C44, C49, C50: 82µF, Capacitor_SMD:C_0402_1005Metric, symbol Device:C_Polarized_Small_US
- added C25, C30, C42, C48, C51, C57: 1µF, Capacitor_SMD:C_0402_1005Metric, symbol Device:C
- added C26, C27, C28, C31, C32, C33, C52, C53, C54, C58, C59, C60: 22µF, Capacitor_SMD:C_0402_1005Metric, symbol Device:C
- added C29, C34, C55, C61: 270µF, Capacitor_SMD:C_0402_1005Metric, symbol Device:C_Polarized_Small_US
- added C35, C36, C56, C62: 1mF, Capacitor_SMD:C_0402_1005Metric, symbol Device:C
- added C37, C38, C63, C64: 4.7µF, Capacitor_SMD:C_0402_1005Metric, symbol Device:C
- added L3, L4: 4.7µH, Inductor_SMD:L_0402_1005Metric, symbol Device:L
- added R10, R12, R18, R20: 48.7k, Resistor_SMD:R_0402_1005Metric, symbol Device:R
- added R11, R13, R19, R21: 301, Resistor_SMD:R_0402_1005Metric, symbol Device:R
- added R17, R8, R9: 100k, Resistor_SMD:R_0402_1005Metric, symbol Device:R
- added R6, R7: 221k, Resistor_SMD:R_0402_1005Metric, symbol Device:R
- added U10, U11, U12, U9: TPS552892RYQR, Package_TO_SOT_SMD:CONV_TPS552892RYQR, symbol Regulator_Switching:TPS552892RYQR
- C13: value 10nF -> 100nF; footprint (none) -> Capacitor_SMD:C_0402_1005Metric
- C15, C16: value C -> 100nF; footprint (none) -> Capacitor_SMD:C_0402_1005Metric
- C18: value nF -> 1µF; footprint (none) -> Capacitor_SMD:C_0402_1005Metric
- C20: value C -> 1µF; footprint (none) -> Capacitor_SMD:C_0402_1005Metric
- L1: footprint (none) -> Inductor_SMD:L_0402_1005Metric
- L2: value 3.6µH -> 4.7µH; footprint (none) -> Inductor_SMD:L_0402_1005Metric
- R14: value 1kR -> 221k; footprint (none) -> Resistor_SMD:R_0402_1005Metric
- R15: value 1.54k -> 221k; footprint (none) -> Resistor_SMD:R_0402_1005Metric
- R16: value 1kR -> 100k; footprint (none) -> Resistor_SMD:R_0402_1005Metric
Connections:
- net BATT_V: now also C18.1, R14.1, R15.1, C17.1, C19.1, C21.1, C22.1, C23.1, C24.1, C41.1, C42.1, C43.1, C44.1, C47.1, C48.1, C49.1, C50.1, R6.1, R7.1, U10.7 (VIN), U11.7 (VIN), U12.7 (VIN), U9.7 (VIN); no longer C15.1, C16.1
- net GND: now also C18.2, C17.2, C19.2, C21.2, C22.2, C23.2, C24.2, C25.2, C26.2, C27.2, C28.2, C29.2, C30.2, C31.2, C32.2, C33.2, C34.2, C37.2, C38.2, C41.2, C42.2, C43.2, C44.2, C47.2, C48.2, C49.2, C50.2, C51.2, C52.2, C53.2, C54.2, C55.2, C57.2, C58.2, C59.2, C60.2, C61.2, C63.2, C64.2, R10.2, R11.2, R12.2, R13.2, R17.2, R18.2, R19.2, R20.2, R21.2, R8.2, R9.2, U10.17 (AGND), U10.2 (MODE), U10.5 (DITH/SYNC), U10.9 (PGND), U11.17 (AGND), U11.2 (MODE), U11.5 (DITH/SYNC), U11.9 (PGND), U12.17 (AGND), U12.2 (MODE), U12.5 (DITH/SYNC), U12.9 (PGND), U9.17 (AGND), U9.2 (MODE), U9.5 (DITH/SYNC), U9.9 (PGND); no longer C15.2, C16.2, R14.2
- net at L2.1: now also C14.2, U10.8 (SW1); no longer C18.2
- net at C13.2, L1.1: now also U9.8 (SW1)
- net at C13.1: now also U9.20 (BOOT1)
- net at R15.2: now also R17.1, U12.1 (EN/UVLO); no longer R14.1
- removed net +3.3V: L1.2, L2.2, R15.1, R16.1
- new net: C45.1, U12.20 (BOOT1)
- new net: C45.2, L4.1, U12.8 (SW1)
- new net: C38.1, U10.18 (VCC), U10.21 (EXTVCC)
- new net: R7.2, R9.1, U10.1 (EN/UVLO)
- new net: C16.2, L2.2, U10.10 (SW2)
- new net: C36.1, U10.15 (COMP)
- new net: C16.1, U10.19 (BOOT2)
- new net: C14.1, U10.20 (BOOT1)
- new net: R12.1, U10.6 (FSW)
- new net: C46.2, L4.2, U12.10 (SW2)
- new net: R6.2, R8.1, U9.1 (EN/UVLO)
- new net: C15.2, L1.2, U9.10 (SW2)
- new net: C35.1, U9.15 (COMP)
- new net: C37.1, U9.18 (VCC), U9.21 (EXTVCC)
- new net: C15.1, U9.19 (BOOT2)
- new net: R10.1, U9.6 (FSW)
- new net: C56.1, U11.15 (COMP)
- new net: C56.2, R19.1
- new net: C39.2, L3.1, U11.8 (SW1)
- new net: C40.2, L3.2, U11.10 (SW2)
- new net: C39.1, U11.20 (BOOT1)
- new net: C63.1, U11.18 (VCC), U11.21 (EXTVCC)
- new net: R14.2, R16.1, U11.1 (EN/UVLO)
- new net: R20.1, U12.6 (FSW)
- new net: C36.2, R13.1
- new net: R18.1, U11.6 (FSW)
- new net: C40.1, U11.19 (BOOT2)
- new net: C62.1, U12.15 (COMP)
- new net: C62.2, R21.1
- new net: C46.1, U12.19 (BOOT2)
- new net: C35.2, R11.1
- new net: C64.1, U12.18 (VCC), U12.21 (EXTVCC)
- new net +5V: C30.1, C31.1, C32.1, C33.1, C34.1, U10.11 (VOUT), U10.12 (ISP), U10.13 (ISN)
- new net +5VM1: C51.1, C52.1, C53.1, C54.1, C55.1, U11.11 (VOUT), U11.12 (ISP), U11.13 (ISN)
- new net +5VM2: C25.1, C26.1, C27.1, C28.1, C29.1, U9.11 (VOUT), U9.12 (ISP), U9.13 (ISN)
- new net +5VM3: C57.1, C58.1, C59.1, C60.1, C61.1, U12.11 (VOUT), U12.12 (ISP), U12.13 (ISN)
- no-connect marks 2 -> 16
