File: PCB_Project/spiSensors.kicad_sch (KiCad schematic)
At the start: 10 parts

Commit message: need to fix the one damn footprint
Parts:
- removed C6, C7: 100nF, Capacitor_SMD:C_0402_1005Metric, symbol Device:C
- removed U3: ~, Package_LGA:LGA-14_3x2.5mm_P0.5mm_LayoutBorder3x4y, symbol Sensor_Motion:ISM330DHCXTR_
Connections:
- no-connect marks 8 -> 6
Other:
- note removed: "ISM330DHCXTR Accelerometer and Gyroscope"

Commit message: re commit
Parts:
- removed C1: 10nF, Capacitor_SMD:C_0402_1005Metric, symbol Device:C
- removed C2: 0.1uF, Capacitor_SMD:C_0402_1005Metric, symbol Device:C
- removed C3: 2.2uF, Capacitor_SMD:C_0402_1005Metric, symbol Device:C
- removed U1: ~, symbol Sensor_Motion:ICM-40609-D
Connections:
- no-connect marks 6 -> 4
Other:
- note removed: "ICM-40609-D Accelerometer and Gyroscope"
- moved on the sheet: C4, C5, U2

Commit message: working on final board
Parts:
- added C10, C12: 100nF, Capacitor_SMD:C_0402_1005Metric, symbol Device:C
- added U8: ~, Sensor:PQFN50P450X300X100-16N, symbol Sensor_Motion:BMI088
- U7: renamed from U2; footprint Sensor:QFN_BMI085_BOS -> Sensor:PQFN50P450X300X100-16N
- renumbered C4 to C11, C5 to C9
Connections:
- net +3V3: now also C10.1, C12.1, U8.11 (VDDIO), U8.3 (VDD)
- net GND: now also C10.2, C12.2, U8.2 (NC), U8.4 (GND), U8.6 (GNDIO), U8.7 (PS)
- net BMI088_INT1_1: now reaches U7.16 (INT1)
- net CSB_Accel_BMI088 renamed CSB_Accel_BMI088_1
- net CSB_Gryo_BMI088 renamed CSB_Gryo_BMI088_1
- net SDI_1 renamed MOSI_1
- net SDO_1 renamed MISO_1
- new net BMI088_INT1_2: U8.16 (INT1)
- new net CSB_Accel_BMI088_2: U8.14 (CSB1)
- new net CSB_Gryo_BMI088_2: U8.5 (CSB2)
- new net MISO_2: U8.10 (SDO2), U8.15 (SDO1)
- new net MOSI_2: U8.9 (SDI)
- new net SCK_2: U8.8 (SCK)
- no-connect marks 4 -> 6
Other:
- moved on the sheet: C11, C9, U7

Commit message: power baby
Parts:
- renumbered C11 to C10, C12 to C11, C9 to C8, C10 to C9
Changed lines of the file:
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@@
+	)
+	(junction
+		(at 135.89 101.6)
+		(diameter 0)
+		(color 0 0 0 0)
 	)
 	(junction
@@
 	(wire
 		(pts
+			(xy 135.89 101.6) (xy 135.89 102.87)
+		)
+		(stroke
+			(width 0)
+			(type default)
+		)
+	)
+	(wire
+		(pts
 			(xy 226.06 90.17) (xy 248.92 90.17)
 		)
@@
 	(wire
 		(pts
-			(xy 128.27 101.6) (xy 130.81 101.6)
+			(xy 128.27 101.6) (xy 135.89 101.6)
 		)
 		(stroke
@@
 	(wire
 		(pts
-			(xy 135.89 97.79) (xy 135.89 102.87)
+			(xy 135.89 97.79) (xy 135.89 101.6)
 		)
 		(stroke
@@
 	(wire
 		(pts
-			(xy 130.81 101.6) (xy 130.81 102.87)
-		)
-		(stroke
-			(width 0)
-			(type default)
-		)
-	)
-	(wire
-		(pts
 			(xy 135.89 102.87) (xy 135.89 105.41)
 		)
@@
 		(pts
 			(xy 233.68 97.79) (xy 233.68 102.87)
-		)
-		(stroke
-			(width 0)
-			(type default)
-		)
-	)
-	(wire
-		(pts
-			(xy 130.81 102.87) (xy 135.89 102.87)
 		)
 		(stroke
@@
 		(dnp no)
 		(fields_autoplaced yes)
-		(property "Reference" "#PWR034"
+		(property "Reference" "#PWR035"
 			(at 248.92 73.66 0)
 			(effects
@@
 			(project "PCB_Project"
 				(path "/3dbd20c6-0b48-4a74-89bd-dd4c54711bfb/8bc0df3c-ce7a-49b1-846c-8bbeab3041e5"
-					(reference "#PWR034")
+					(reference "#PWR035")
 					(unit 1)
 				)
@@
 		(on_board yes)
 		(dnp no)
-		(property "Reference" "#PWR040"
+		(property "Reference" "#PWR041"
 			(at 96.52 110.49 0)
 			(effects
@@
 			(project "PCB_Project"
 				(path "/3dbd20c6-0b48-4a74-89bd-dd4c54711bfb/8bc0df3c-ce7a-49b1-846c-8bbeab3041e5"
-					(reference "#PWR040")
+					(reference "#PWR041")
 					(unit 1)
 				)
@@
 		(dnp no)
 		(fields_autoplaced yes)
-		(property "Reference" "#PWR042"
+		(property "Reference" "#PWR043"
 			(at 135.89 111.76 0)
 			(effects
@@
 			(project "PCB_Project"
 				(path "/3dbd20c6-0b48-4a74-89bd-dd4c54711bfb/8bc0df3c-ce7a-49b1-846c-8bbeab3041e5"
-					(reference "#PWR042")
+					(reference "#PWR043")
 					(unit 1)
 				)
@@
 		(dnp no)
 		(fields_autoplaced yes)
-		(property "Reference" "#PWR037"
+		(property "Reference" "#PWR038"
 			(at 248.92 90.17 0)
 			(effects
@@
 			(project "PCB_Project"
 				(path "/3dbd20c6-0b48-4a74-89bd-dd4c54711bfb/8bc0df3c-ce7a-49b1-846c-8bbeab3041e5"
-					(reference "#PWR037")
+					(reference "#PWR038")
 					(unit 1)
 				)
@@
 		(on_board yes)
 		(dnp no)
-		(property "Reference" "C11"
+		(property "Reference" "C10"
 			(at 143.51 96.52 0)
 			(effects
@@
 			(project "PCB_Project"
 				(path "/3dbd20c6-0b48-4a74-89bd-dd4c54711bfb/8bc0df3c-ce7a-49b1-846c-8bbeab3041e5"
-					(reference "C11")
+					(reference "C10")
 					(unit 1)
 				)
@@
 		(dnp no)
 		(fields_autoplaced yes)
-		(property "Reference" "#PWR036"
+		(property "Reference" "#PWR037"
 			(at 151.13 90.17 0)
 			(effects
@@
 			(project "PCB_Project"
 				(path "/3dbd20c6-0b48-4a74-89bd-dd4c54711bfb/8bc0df3c-ce7a-49b1-846c-8bbeab3041e5"
-					(reference "#PWR036")
+					(reference "#PWR037")
 					(unit 1)
 				)
@@
 		(dnp no)
 		(fields_autoplaced yes)
-		(property "Reference" "#PWR035"
+		(property "Reference" "#PWR036"
 			(at 151.13 74.93 0)
 			(effects
@@
 			(project "PCB_Project"
 				(path "/3dbd20c6-0b48-4a74-89bd-dd4c54711bfb/8bc0df3c-ce7a-49b1-846c-8bbeab3041e5"
-					(reference "#PWR035")
+					(reference "#PWR036")
 					(unit 1)
 				)
@@
 		(dnp no)
 		(fields_autoplaced yes)
-		(property "Reference" "C10"
+		(property "Reference" "C9"
 			(at 252.73 85.0899 0)
 			(effects
@@
 			(project "PCB_Project"
 				(path "/3dbd20c6-0b48-4a74-89bd-dd4c54711bfb/8bc0df3c-ce7a-49b1-846c-8bbeab3041e5"
-					(reference "C10")
+					(reference "C9")
 					(unit 1)
 				)
@@
 		(on_board yes)
 		(dnp no)
-		(property "Reference" "#PWR041"
+		(property "Reference" "#PWR042"
 			(at 194.31 110.49 0)
 			(effects
@@
 			(project "PCB_Project"
 				(path "/3dbd20c6-0b48-4a74-89bd-dd4c54711bfb/8bc0df3c-ce7a-49b1-846c-8bbeab3041e5"
-					(reference "#PWR041")
+					(reference "#PWR042")
 					(unit 1)
 				)
@@
 		(dnp no)
 		(fields_autoplaced yes)
-		(property "Reference" "C9"
+		(property "Reference" "C8"
 			(at 154.94 85.0899 0)
 			(effects
@@
 			(project "PCB_Project"
 				(path "/3dbd20c6-0b48-4a74-89bd-dd4c54711bfb/8bc0df3c-ce7a-49b1-846c-8bbeab3041e5"
-					(reference "C9")
+					(reference "C8")
 					(unit 1)
 				)
@@
 		(on_board yes)
 		(dnp no)
-		(property "Reference" "#PWR039"
+		(property "Reference" "#PWR040"
 			(at 237.49 93.98 0)
 			(effects
@@
 			(project "PCB_Project"
 				(path "/3dbd20c6-0b48-4a74-89bd-dd4c54711bfb/8bc0df3c-ce7a-49b1-846c-8bbeab3041e5"
-					(reference "#PWR039")
+					(reference "#PWR040")
 					(unit 1)
 				)
@@
 		(dnp no)
 		(fields_autoplaced yes)
-		(property "Reference" "#PWR043"
+		(property "Reference" "#PWR044"
 			(at 233.68 111.76 0)
 			(effects
@@
 			(project "PCB_Project"
 				(path "/3dbd20c6-0b48-4a74-89bd-dd4c54711bfb/8bc0df3c-ce7a-49b1-846c-8bbeab3041e5"
-					(reference "#PWR043")
+					(reference "#PWR044")
 					(unit 1)
 				)
@@
 		(on_board yes)
 		(dnp no)
-		(property "Reference" "#PWR038"
+		(property "Reference" "#PWR039"
 			(at 139.7 93.98 0)
 			(effects
@@
 			(project "PCB_Project"
 				(path "/3dbd20c6-0b48-4a74-89bd-dd4c54711bfb/8bc0df3c-ce7a-49b1-846c-8bbeab3041e5"
-					(reference "#PWR038")
+					(reference "#PWR039")
 					(unit 1)
 				)
@@
 		(on_board yes)
 		(dnp no)
-		(property "Reference" "C12"
+		(property "Reference" "C11"
 			(at 241.3 96.52 0)
 			(effects
@@
 			(project "PCB_Project"
 				(path "/3dbd20c6-0b48-4a74-89bd-dd4c54711bfb/8bc0df3c-ce7a-49b1-846c-8bbeab3041e5"
-					(reference "C12")
+					(reference "C11")
 					(unit 1)
 				)

Commit message: finally
Changed lines of the file:
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@@
+		)
+	)
+	(text_box "high freq ceramic for C's"
+		(exclude_from_sim no)
+		(at 149.86 116.84 0)
+		(size 27.94 3.175)
+		(stroke
+			(width 0)
+			(type default)
+		)
+		(fill
+			(type none)
+		)
+		(effects
+			(font
+				(size 1.27 1.27)
+			)
+			(justify left top)
 		)
 	)
