File: Power Distribution/Power Distribution.kicad_sch (KiCad schematic)
At the start: 81 parts, among them J1 Batt_Connector, J2 Motor Connector 1, J3 Motor Connector 2, J4 Motor Connector 3, J5 Motor Connector 3, U1 TPS552892RYQR, U2 TPS552892RYQR, U3 TPS552892RYQR, U4 TPS552892RYQR

Commit message: added fabs and fixed i2c loop
Parts:
- removed C1, C2, C27, C28, C3, C33, C34, C4: 100nF, Capacitor_SMD:C_0402_1005Metric, symbol Device:C
- removed C10, C11, C12, C31, C32, C37, C38, C9: 82µF, Capacitor_THT:CP_Radial_D10.0mm_P5.00mm, symbol Device:C_Polarized_Small_US
- removed C13, C18, C30, C36, C39, C45, C6, C8: 1µF, Capacitor_SMD:C_0402_1005Metric, symbol Device:C
- removed C14, C15, C16, C19, C20, C21, C40, C41, C42, C46, C47, C48: 22µF, Capacitor_SMD:C_0603_1608Metric, symbol Device:C
- removed C17, C22, C43, C49: 270µF, Capacitor_THT:CP_Radial_D6.3mm_P2.50mm, symbol Device:C_Polarized_Small_US
- removed C23, C24, C44, C50: 56nF, Capacitor_SMD:C_0603_1608Metric, symbol Device:C
- removed C25, C26, C51, C52: 4.7µF, Capacitor_SMD:C_0402_1005Metric, symbol Device:C
- removed C29, C35: 10µF, Capacitor_SMD:C_0603_1608Metric, symbol Device:C
- removed C5, C7: 10µF, Capacitor_SMD:C_0402_1005Metric, symbol Device:C
- removed L1, L2, L3, L4: 4.7µH, Inductor_SMD:L_Changjiang_FNR252010S, symbol Device:L
- removed R1, R10, R2, R9: 221k, Resistor_SMD:R_1206_3216Metric, symbol Device:R
- removed R11, R12, R3, R4: 100k, Resistor_SMD:R_0603_1608Metric, symbol Device:R
- removed R13, R15, R5, R7: 48.7k, Resistor_SMD:R_1206_3216Metric, symbol Device:R
- removed R14, R16, R6, R8: 301, Resistor_SMD:R_0603_1608Metric, symbol Device:R
- removed U1, U2, U3, U4: TPS552892RYQR, Package_TO_SOT_SMD:CONV_TPS552892RYQR, symbol Regulator_Switching:TPS552892RYQR
Connections:
- no-connect marks 16 -> 0
